Commit message: Harmonic
Signed-off-by: Juancams <jc.manzanares.serrano@gmail.com>

File: pmb2_description/ros2_control/ros2_control.urdf.xacro (robot description, xacro)
@@ -21,5 +21,5 @@
     <xacro:if value="${use_sim_time}">
       <gazebo>
-        <plugin filename="libgazebo_ros2_control.so" name="gazebo_ros2_control">
+        <plugin filename="libgz_ros2_control-system.so" name="gz_ros2_control::GazeboSimROS2ControlPlugin">
           <parameters>$(find pmb2_description)/ros2_control/gazebo_controller_manager_cfg.yaml</parameters>
         </plugin>
@@ -32,5 +32,5 @@
         <!-- HW interface gazebo-->
         <hardware>
-          <plugin>gazebo_ros2_control/GazeboSystem</plugin>
+          <plugin>gz_ros2_control/GazeboSimSystem</plugin>
         </hardware>
         <!-- IMU sensor (only in simulation)-->

File: pmb2_description/urdf/base/base.gazebo.xacro (robot description, xacro)
@@ -31,5 +31,5 @@
     </gazebo>
     <!-- Odometry plugin for ground truth -->
-    <gazebo>
+    <!-- <gazebo>
       <plugin filename="libgazebo_world_odometry.so" name="gazebo_ros_odometry">
         <frame_name>world</frame_name>
@@ -41,5 +41,5 @@
         </xacro:if>
       </plugin>
-    </gazebo>
+    </gazebo> -->
   </xacro:macro>
 </robot>

File: pmb2_description/urdf/base/base.urdf.xacro (robot description, xacro)
@@ -46,5 +46,5 @@
         <origin xyz="0 0 0" rpy="0 0 0" />
         <geometry>
-          <mesh filename="package://pmb2_description/meshes/base/base.stl" />
+          <mesh filename="file://$(find pmb2_description)/meshes/base/base.stl" />
         </geometry>
         <material name="White" />
@@ -53,5 +53,5 @@
         <origin xyz="0 0 0" rpy="0 0 0" />
         <geometry>
-          <mesh filename="package://pmb2_description/meshes/base/high_resolution/base_collision.stl" />
+          <mesh filename="file://$(find pmb2_description)/meshes/base/high_resolution/base_collision.stl" />
         </geometry>
         <material name="White" />

File: pmb2_description/urdf/cameras_add_on/cameras_add_on.urdf.xacro (robot description, xacro)
@@ -26,5 +26,5 @@
         <origin xyz="0 0 0" rpy="0 0 0"/>
         <geometry>
-          <mesh filename="package://pmb2_description/meshes/cameras_add_on/cameras_add_on.stl" scale="1 1 1"/>
+          <mesh filename="file://$(find pmb2_description)/meshes/cameras_add_on/cameras_add_on.stl" scale="1 1 1"/>
         </geometry>
         <material name="White" />
@@ -33,5 +33,5 @@
         <origin xyz="0 0 0" rpy="0 0 0" />
         <geometry>
-          <mesh filename="package://pmb2_description/meshes/cameras_add_on/cameras_add_on_collision.stl" scale="1 1 1"/>
+          <mesh filename="file://$(find pmb2_description)/meshes/cameras_add_on/cameras_add_on_collision.stl" scale="1 1 1"/>
         </geometry>
         <material name="White" />

File: pmb2_description/urdf/dock/dock.urdf.xacro (robot description, xacro)
@@ -27,5 +27,5 @@
         <origin xyz="0 0 0" rpy="0 0 0" />
         <geometry>
-          <mesh filename="package://pmb2_description/meshes/dock/dock.stl" />
+          <mesh filename="file://$(find pmb2_description)/meshes/dock/dock.stl" />
         </geometry>
         <material name="LightGrey" />
@@ -34,5 +34,5 @@
         <origin xyz="0 0 0" rpy="0 0 0" />
         <geometry>
-          <mesh filename="package://pmb2_description/meshes/dock/dock_collision.stl" />
+          <mesh filename="file://$(find pmb2_description)/meshes/dock/dock_collision.stl" />
         </geometry>
         <material name="LightGrey" />

File: pmb2_description/urdf/objects/antenna.urdf.xacro (robot description, xacro)
@@ -24,5 +24,5 @@
         <origin xyz="0 0 0" rpy="0 0 0"/>
         <geometry>
-          <mesh filename="package://pmb2_description/meshes/objects/antenna.stl"/>
+          <mesh filename="file://$(find pmb2_description)/meshes/objects/antenna.stl"/>
         </geometry>
         <material name="Black"/>

File: pmb2_description/urdf/objects/cover.urdf.xacro (robot description, xacro)
@@ -24,5 +24,5 @@
         <origin xyz="0 0 0" rpy="0 0 0"/>
         <geometry>
-          <mesh filename="package://pmb2_description/meshes/base/base_ring.stl"/>
+          <mesh filename="file://$(find pmb2_description)/meshes/base/base_ring.stl"/>
         </geometry>
         <material name="Orange"/>

File: pmb2_description/urdf/sensors/bumper.urdf.xacro (robot description, xacro)
@@ -24,5 +24,5 @@
         <origin xyz="0 0 0" rpy="0 0 0" />
         <geometry>
-          <mesh filename="package://pmb2_description/meshes/sensors/bumper.stl"/>
+          <mesh filename="file://$(find pmb2_description)/meshes/sensors/bumper.stl"/>
         </geometry>
         <material name="DarkGrey"/>
@@ -31,5 +31,5 @@
         <origin xyz="0 0 0" rpy="0 0 0" />
         <geometry>
-          <mesh filename="package://pmb2_description/meshes/sensors/bumper_collision.stl"/>
+          <mesh filename="file://$(find pmb2_description)/meshes/sensors/bumper_collision.stl"/>
         </geometry>
         <material name="DarkGrey"/>

File: pmb2_description/urdf/sensors/elp_rgb.gazebo.xacro (robot description, xacro)
@@ -35,5 +35,5 @@
           </noise>
         </camera>
-        <plugin name="${name}_frame_controller" filename="libgazebo_ros_camera.so">
+        <!-- <plugin name="${name}_frame_controller" filename="libgazebo_ros_camera.so">
           <alwaysOn>true</alwaysOn>
           <updateRate>0.0</updateRate>
@@ -47,5 +47,5 @@
           <distortionT1>0.0</distortionT1>
           <distortionT2>0.0</distortionT2>
-        </plugin>
+        </plugin> -->
       </sensor>
     </gazebo>

File: pmb2_description/urdf/sensors/elp_rgb.urdf.xacro (robot description, xacro)
@@ -32,5 +32,5 @@
         <origin xyz="0 0 0" rpy="0 90 0"/>
         <geometry>
-          <mesh filename="package://pmb2_description/meshes/sensors/elp_camera.stl" scale="0.001 0.001 0.001"/>
+          <mesh filename="file://$(find pmb2_description)/meshes/sensors/elp_camera.stl" scale="0.001 0.001 0.001"/>
         </geometry>
         <material name="Grey" />

File: pmb2_description/urdf/sensors/hokuyo_urg_04lx_ug01_laser.gazebo.xacro (robot description, xacro)
@@ -15,9 +15,11 @@
   <xacro:macro name="hokuyo_urg_04lx_ug01_laser_gazebo" params="name ros_topic update_rate min_angle max_angle">
     <gazebo reference="${name}_link">
-      <sensor type="ray" name="${name}">
+      <sensor type="lidar" name="${name}">
         <pose>0 0 0 0 0 0</pose>
         <update_rate>${update_rate}</update_rate>
         <visualize>true</visualize>
-        <ray>
+        <topic>${ros_topic}</topic>
+        <gz_frame_id>${name}_link</gz_frame_id>
+        <lidar>
           <scan>
             <horizontal>
@@ -39,12 +41,5 @@
             <stddev>0.03</stddev>
           </noise>
-        </ray>
-        <plugin name="${name}" filename="libgazebo_ros_ray_sensor.so">
-          <ros>
-            <remapping>~/out:=${ros_topic}</remapping>
-          </ros>
-          <output_type>sensor_msgs/LaserScan</output_type>
-          <frame_name>${name}_link</frame_name>
-        </plugin>
+        </lidar>
       </sensor>
       <material>Gazebo/DarkGrey</material>

File: pmb2_description/urdf/sensors/hokuyo_urg_04lx_ug01_laser.urdf.xacro (robot description, xacro)
@@ -24,5 +24,5 @@
         <origin xyz="0 0 0" rpy="0 0 0" />
         <geometry>
-          <mesh filename="package://pmb2_description/meshes/sensors/hokuyo_urg_04lx_ug01.stl"/>
+          <mesh filename="file://$(find pmb2_description)/meshes/sensors/hokuyo_urg_04lx_ug01.stl"/>
         </geometry>
         <material name="DarkGrey"/>

File: pmb2_description/urdf/sensors/range.gazebo.xacro (robot description, xacro)
@@ -15,9 +15,11 @@
   <xacro:macro name="range_gazebo" params="name ros_topic update_rate maxRange minRange fov radiation">
     <gazebo reference="${name}_link">
-      <sensor type="ray" name="${name}">
+      <sensor type="lidar" name="${name}">
         <pose>0 0 0 0 0 0</pose>
         <update_rate>${update_rate}</update_rate>
         <visualize>false</visualize>
-        <ray>
+        <topic>${ros_topic}</topic>
+        <gz_frame_id>${name}_link</gz_frame_id>
+        <lidar>
           <scan>
             <horizontal>
@@ -44,14 +46,5 @@
             <stddev>0.005</stddev>
           </noise>
-        </ray>
-        <plugin name="${name}_gazebo_ros_range" filename="libgazebo_ros_ray_sensor.so">
-          <ros>
-            <namespace></namespace>
-            <remapping>~/out:=${ros_topic}</remapping>
-          </ros>
-          <output_type>sensor_msgs/Range</output_type>
-          <radiation_type>${radiation}</radiation_type>
-          <frame_name>${name}_link</frame_name>
-        </plugin>
+        </lidar>
       </sensor>
       <material>Gazebo/DarkGrey</material>

File: pmb2_description/urdf/sensors/range.urdf.xacro (robot description, xacro)
@@ -24,5 +24,5 @@
         <origin xyz="0 0 0" rpy="0 0 0" />
         <geometry>
-          <mesh filename="package://pmb2_description/meshes/sensors/srf05.stl"/>
+          <mesh filename="file://$(find pmb2_description)/meshes/sensors/srf05.stl"/>
         </geometry>
         <material name="DarkGrey"/>

File: pmb2_description/urdf/sensors/sick_tim551_laser.gazebo.xacro (robot description, xacro)
@@ -15,9 +15,11 @@
   <xacro:macro name="sick_tim551_laser_gazebo" params="name ros_topic update_rate min_angle max_angle">
     <gazebo reference="${name}_link">
-      <sensor type="ray" name="${name}">
+      <sensor type="lidar" name="${name}">
         <pose>0 0 0 0 0 0</pose>
         <update_rate>${update_rate}</update_rate>
         <visualize>true</visualize>
-        <ray>
+        <topic>${ros_topic}</topic>
+        <gz_frame_id>${name}_link</gz_frame_id>
+        <lidar>
           <scan>
             <horizontal>
@@ -39,12 +41,5 @@
             <stddev>0.01</stddev>
           </noise>
-        </ray>
-        <plugin name="${name}" filename="libgazebo_ros_ray_sensor.so">
-          <ros>
-            <remapping>~/out:=${ros_topic}</remapping>
-          </ros>
-          <output_type>sensor_msgs/LaserScan</output_type>
-          <frame_name>${name}_link</frame_name>
-        </plugin>
+        </lidar>
       </sensor>
       <material>Gazebo/DarkGrey</material>

File: pmb2_description/urdf/sensors/sick_tim551_laser.urdf.xacro (robot description, xacro)
@@ -24,5 +24,5 @@
         <origin xyz="0 0 0" rpy="0 0 0" />
         <geometry>
-          <mesh filename="package://pmb2_description/meshes/sensors/sick_tim551.stl"/>
+          <mesh filename="file://$(find pmb2_description)/meshes/sensors/sick_tim551.stl"/>
         </geometry>
         <material name="DarkGrey"/>

File: pmb2_description/urdf/sensors/sick_tim561_laser.gazebo.xacro (robot description, xacro)
@@ -15,9 +15,11 @@
   <xacro:macro name="sick_tim561_laser_gazebo" params="name ros_topic update_rate min_angle max_angle">
     <gazebo reference="${name}_link">
-      <sensor type="ray" name="${name}">
+      <sensor type="lidar" name="${name}">
         <pose>0 0 0 0 0 0</pose>
         <update_rate>${update_rate}</update_rate>
         <visualize>true</visualize>
-        <ray>
+        <topic>${ros_topic}</topic>
+        <gz_frame_id>${name}_link</gz_frame_id>
+        <lidar>
           <scan>
             <horizontal>
@@ -39,12 +41,5 @@
             <stddev>0.01</stddev>
           </noise>
-        </ray>
-        <plugin name="${name}" filename="libgazebo_ros_ray_sensor.so">
-          <ros>
-            <remapping>~/out:=${ros_topic}</remapping>
-          </ros>
-          <output_type>sensor_msgs/LaserScan</output_type>
-          <frame_name>${name}_link</frame_name>
-        </plugin>
+        </lidar>
       </sensor>
       <material>Gazebo/DarkGrey</material>

File: pmb2_description/urdf/sensors/sick_tim561_laser.urdf.xacro (robot description, xacro)
@@ -24,5 +24,5 @@
         <origin xyz="0 0 0" rpy="0 0 0" />
         <geometry>
-          <mesh filename="package://pmb2_description/meshes/sensors/sick_tim551.stl"/>
+          <mesh filename="file://$(find pmb2_description)/meshes/sensors/sick_tim551.stl"/>
         </geometry>
         <material name="DarkGrey"/>

File: pmb2_description/urdf/sensors/sick_tim571_laser.gazebo.xacro (robot description, xacro)
@@ -15,9 +15,11 @@
   <xacro:macro name="sick_tim571_laser_gazebo" params="name ros_topic update_rate min_angle max_angle">
     <gazebo reference="${name}_link">
-      <sensor type="ray" name="${name}">
+      <sensor type="lidar" name="${name}">
         <pose>0 0 0 0 0 0</pose>
         <update_rate>${update_rate}</update_rate>
         <visualize>true</visualize>
-        <ray>
+        <topic>${ros_topic}</topic>
+        <gz_frame_id>${name}_link</gz_frame_id>
+        <lidar>
           <scan>
             <horizontal>
@@ -39,12 +41,5 @@
             <stddev>0.01</stddev>
           </noise>
-        </ray>
-        <plugin name="${name}" filename="libgazebo_ros_ray_sensor.so">
-          <ros>
-            <remapping>~/out:=${ros_topic}</remapping>
-          </ros>
-          <output_type>sensor_msgs/LaserScan</output_type>
-          <frame_name>${name}_link</frame_name>
-        </plugin>
+        </lidar>
       </sensor>
       <material>Gazebo/DarkGrey</material>

File: pmb2_description/urdf/sensors/sick_tim571_laser.urdf.xacro (robot description, xacro)
@@ -24,5 +24,5 @@
         <origin xyz="0 0 0" rpy="0 0 0" />
         <geometry>
-          <mesh filename="package://pmb2_description/meshes/sensors/sick_tim551.stl"/>
+          <mesh filename="file://$(find pmb2_description)/meshes/sensors/sick_tim551.stl"/>
         </geometry>
         <material name="DarkGrey"/>
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