Commit message: Fix Tiago lidar sensor 571
Signed-off-by: Francisco Martín Rico <fmrico@gmail.com>

File: pmb2_description/urdf/sensors/sick_tim571_laser.gazebo.xacro (robot description, xacro)
@@ -15,8 +15,8 @@
   <xacro:macro name="sick_tim571_laser_gazebo" params="name ros_topic update_rate min_angle max_angle">
     <gazebo reference="${name}_link">
-      <sensor type="lidar" name="${name}">
-        <pose>0 0 0 0 0 0</pose>
+      <sensor type="gpu_lidar" name="sick_tim571">
         <update_rate>${update_rate}</update_rate>
         <visualize>true</visualize>
+        <always_on>true</always_on>
         <topic>${ros_topic}</topic>
         <gz_frame_id>${name}_link</gz_frame_id>
@@ -43,5 +43,4 @@
         </lidar>
       </sensor>
-      <material>Gazebo/DarkGrey</material>
     </gazebo>
   </xacro:macro>

File: pmb2_description/urdf/sensors/sick_tim571_laser.urdf.xacro (robot description, xacro)
@@ -15,5 +15,5 @@
   <xacro:include filename="$(find pmb2_description)/urdf/sensors/sick_tim571_laser.gazebo.xacro" />
   <xacro:macro name="sick_tim571_laser" params="name parent *origin ros_topic update_rate min_angle max_angle">
-    <link name="${name}_link" type="laser">
+    <link name="${name}_link">
       <inertial>
         <origin xyz="-0.02559000000 -0.00056000000 -0.05732000000" rpy="0 0 0"/>
@@ -22,5 +22,4 @@
       </inertial>
       <visual>
-        <origin xyz="0 0 0" rpy="0 0 0" />
         <geometry>
           <mesh filename="file://$(find pmb2_description)/meshes/sensors/sick_tim551.stl"/>
