Commit message: Changed laser position
Signed-off-by: Juancams <jc.manzanares.serrano@gmail.com>

File: pmb2_description/urdf/base/base_sensors.urdf.xacro (robot description, xacro)
@@ -14,5 +14,5 @@
 <robot xmlns:xacro="http://ros.org/wiki/xacro">
   <!-- PROPERTIES -->
-  <xacro:property name="base_laser_x" value="0.202"/>
+  <xacro:property name="base_laser_x" value="0.252"/>
   <xacro:property name="base_laser_y" value="0.0"/>
   <xacro:property name="base_laser_z" value="-0.004"/>
